File: typec/typec.sch (KiCad schematic (older format))
At the start: 17 parts, among them U1 TPD6E05U06-USON, U2 TPD4E05U06-USON, U3 TPS62081-WSON, U4 TPD4E05U06-USON, U5 TPS74801-VSON

Commit message: Added TUSB212 and USB 3.1 Connector
Parts:
- added C10: 10uf/10v, Capacitor_SMD:C_0805_2012Metric, symbol Device:C
- added C8, C9: 0.1uF/10v, Capacitor_SMD:C_0402_1005Metric, symbol Device:C
- added R5: 1.6K, Resistor_SMD:R_0805_2012Metric, symbol Device:R_Small_US
- added R6: 43K, Resistor_SMD:R_0805_2012Metric, symbol Device:R_Small_US
- added R7, R8: 0 E, Resistor_SMD:R_0805_2012Metric, symbol Device:R_Small_US
- added U6: TUSB212-X2QFN, TUSB212-X2QFN:TUSB212-X2QFN, symbol TUSB212-X2QFN:TUSB212-X2QFN
- added USB1: Wurth-632723300011, Type-C:Wurth-632723300011-MaximumExtensionMount, symbol TYPEC_MODULES:Wurth-632723300011
- U3: symbol TPS62081-WSON:TPS62081-WSON -> typec-rescue:TPS62081-WSON-TPS62081-WSON
- U5: symbol TPS74801-VSON:TPS74801-VSON -> typec-rescue:TPS74801-VSON-TPS74801-VSON
Connections:
- wire segments 79 -> 142
Other:
- moved on the sheet: C1, C2, C3, C4, C5, C6, C7, L1, R1, R2, R3, R4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
