File: typec/Multiplexer.sch (KiCad schematic (older format))
At the start: 19 parts

Commit message: updated
Parts:
- added D6, D7, D8: LED, LED_SMD:LED_0402_1005Metric, symbol Device:LED
- added JP3, JP8, JP9: Jumper_3_Open, Connector_JST:JST_EH_B3B-EH-A_1x03_P2.50mm_Vertical, symbol Jumper:Jumper_3_Open
- added R11: 330 E, Resistor_SMD:R_0402_1005Metric, symbol Device:R_Small_US
- added R19, R22, R25: 200 K, Resistor_SMD:R_0402_1005Metric, symbol Device:R_Small_US
- added R23, R26: 500 E, Resistor_SMD:R_0402_1005Metric, symbol Device:R_Small_US
- added R27: NC / 10 K, Resistor_SMD:R_0402_1005Metric, symbol Device:R_Small_US
- added R28: NC/ 10 K, Resistor_SMD:R_0402_1005Metric, symbol Device:R_Small_US
- added TP3, TP4, TP5: TestPoint, TestPoint:TestPoint_THTPad_2.0x2.0mm_Drill1.0mm, symbol Connector:TestPoint
- C10: renamed from C11; footprint Capacitor_SMD:C_0805_2012Metric -> Capacitor_SMD:C_0603_1608Metric
- C13: renamed from C14; footprint Capacitor_SMD:C_0805_2012Metric -> Capacitor_SMD:C_0402_1005Metric
- R12: renamed from R9; footprint Resistor_SMD:R_0805_2012Metric -> Resistor_SMD:R_0201_0603Metric
- R13: renamed from R10; footprint Resistor_SMD:R_0805_2012Metric -> Resistor_SMD:R_0402_1005Metric
- R14: renamed from R11; footprint Resistor_SMD:R_0805_2012Metric -> Resistor_SMD:R_0402_1005Metric
- R15: renamed from R12; footprint Resistor_SMD:R_0805_2012Metric -> Resistor_SMD:R_0201_0603Metric
- R16: renamed from R13; footprint Resistor_SMD:R_0805_2012Metric -> Resistor_SMD:R_0402_1005Metric
- R17: renamed from R14; footprint Resistor_SMD:R_0805_2012Metric -> Resistor_SMD:R_0402_1005Metric
- R18: renamed from R15; footprint Resistor_SMD:R_0805_2012Metric -> Resistor_SMD:R_0402_1005Metric
- R20: renamed from R16; footprint Resistor_SMD:R_0805_2012Metric -> Resistor_SMD:R_0402_1005Metric
- R21: renamed from R17; footprint Resistor_SMD:R_0805_2012Metric -> Resistor_SMD:R_0201_0603Metric
- renumbered C12 to C11, C13 to C12, C15 to C14, C16 to C15, C17 to C16, C18 to C17
Connections:
- net GND: now also MUX1.31 (GND), D6.1 (K), JP3.1 (A), JP8.1 (A), JP9.1 (A), R28.2; no longer C11.2, C12.2, R16.2, R17.1, R18.1
- net VBUS: now also JP3.3 (B), R19.2, R22.1, R23.1, R25.1, R26.1, R27.1
- net VOUT(3.3V): now also R11.1
- net DIR: now reaches MUX1.11 (DIR)
- net DIR: now also R22.2, TP3.1
- net ADDR: now reaches MUX1.22 (ADDR)
- net ADDR: now also R27.2, R28.1, TP5.1
- net INT_NOUT3: now reaches MUX1.23 (INT_N/OUT3)
- net INT_NOUT3: now also R25.2, TP4.1
- net SDAOUT1: now reaches MUX1.25 (SDA/OUT1)
- net SDAOUT1: now also JP8.2 (C)
- net SCLOUT2: now reaches MUX1.26 (SCL/OUT2)
- net SCLOUT2: now also JP9.2 (C)
- net at MUX1.27 (ID): now also R19.1
- net at MUX1.4 (PORT): now also R16.2; no longer R16.1
- net CC1 renamed CC10
- net CC2 renamed CC20
- net CRX1N renamed CRX1N0
- net CRX1P renamed CRX1P0
- net CRX2N renamed CRX2N0
- net CRX2P renamed CRX2P0
- net CTX1N renamed CTX1N0
- net CTX1P renamed CTX1P0
- net CTX2N renamed CTX2N0
- net CTX2P renamed CTX2P0
- new net: JP3.2 (C), R16.1
- new net: D8.2 (A), R26.2
- new net: D8.1 (K), JP9.3 (B)
- new net: D7.2 (A), R23.2
- new net: D7.1 (K), JP8.3 (B)
- new net: D6.2 (A), R11.2
- new net USB3_RX0N: C11.2, R17.1
- new net USB3_RX0P: C12.2, R18.1
- no-connect marks 7 -> 1
Other:
- moved on the sheet: C10, C11, C12, C13, C14, C15, C16, C17, FB1, MUX1, R12, R13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
