File: typec2.0/_saved_typec2.0.sch (KiCad schematic (older format))
At the start: 75 parts, among them J1 Conn_01x05_Male, J2 Conn_01x05_Female, J3 Conn_01x05_Female, J4 Conn_01x05_Female, J5 Conn_01x05_Female, U1 TUSB2046, U2 TPS2044-SOIC, U3 SN75240PWR, U4 TPS62082-WSON, U5 SN75240PWR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

Commit message: 2.0
Parts:
- removed J3: Conn_01x05_Female, Connector_JST:JST_ACH_BM05B-ACHSS-A-GAN-ETF_1x05-1MP_P1.20mm_Vertical, symbol Connector:Conn_01x05_Female
- added J?: Conn_01x05_Female, Connector_JST:JST_GH_SM05B-GHS-TB_1x05-1MP_P1.25mm_Horizontal, symbol Connector:Conn_01x05_Female
- added TP2: TestPoint, TestPoint:TestPoint_THTPad_2.0x2.0mm_Drill1.0mm, symbol Connector:TestPoint
- J1, J2, J4, J5: footprint Connector_JST:JST_ACH_BM05B-ACHSS-A-GAN-ETF_1x05-1MP_P1.20mm_Vertical -> Connector_JST:JST_GH_SM05B-GHS-TB_1x05-1MP_P1.25mm_Horizontal
Connections:
- net GND: now also J?.4 (Pin_4), J?.5 (Pin_5)
- net VBUS(5V): now also TP2.1
- net VOUT2(5V): now also J?.1 (Pin_1)
- net at R16.1, U6.6 (B): now also J?.2 (Pin_2)
- net at R17.2, U6.8 (A): now also J?.3 (Pin_3)
Changed lines of the file:
@@
 EESchema Schematic File Version 4
-LIBS:typec2.0-cache
 EELAYER 29 0
 EELAYER END
@@
 F 0 "J1" H 808 3031 50  0000 C CNN
 F 1 "Conn_01x05_Male" H 808 2940 50  0000 C CNN
-F 2 "Connector_JST:JST_ACH_BM05B-ACHSS-A-GAN-ETF_1x05-1MP_P1.20mm_Vertical" H 700 2650 50  0001 C CNN
+F 2 "Connector_JST:JST_GH_SM05B-GHS-TB_1x05-1MP_P1.25mm_Horizontal" H 700 2650 50  0001 C CNN
 F 3 "~" H 700 2650 50  0001 C CNN
 	1    700  2650
@@
 F 0 "J2" H 9778 1226 50  0000 L CNN
 F 1 "Conn_01x05_Female" H 9778 1135 50  0000 L CNN
-F 2 "Connector_JST:JST_ACH_BM05B-ACHSS-A-GAN-ETF_1x05-1MP_P1.20mm_Vertical" H 9750 1200 50  0001 C CNN
+F 2 "Connector_JST:JST_GH_SM05B-GHS-TB_1x05-1MP_P1.25mm_Horizontal" H 9750 1200 50  0001 C CNN
 F 3 "~" H 9750 1200 50  0001 C CNN
 	1    9750 1200
-	1    0    0    -1
-$EndComp
-$Comp
-L Connector:Conn_01x05_Female J3
-U 1 1 5D5B9F9F
-P 9850 2600
-F 0 "J3" H 9878 2626 50  0000 L CNN
-F 1 "Conn_01x05_Female" H 9878 2535 50  0000 L CNN
-F 2 "Connector_JST:JST_ACH_BM05B-ACHSS-A-GAN-ETF_1x05-1MP_P1.20mm_Vertical" H 9850 2600 50  0001 C CNN
-F 3 "~" H 9850 2600 50  0001 C CNN
-	1    9850 2600
 	1    0    0    -1
 $EndComp
@@
 F 0 "J4" H 9928 4126 50  0000 L CNN
 F 1 "Conn_01x05_Female" H 9928 4035 50  0000 L CNN
-F 2 "Connector_JST:JST_ACH_BM05B-ACHSS-A-GAN-ETF_1x05-1MP_P1.20mm_Vertical" H 9900 4100 50  0001 C CNN
+F 2 "Connector_JST:JST_GH_SM05B-GHS-TB_1x05-1MP_P1.25mm_Horizontal" H 9900 4100 50  0001 C CNN
 F 3 "~" H 9900 4100 50  0001 C CNN
 	1    9900 4100
@@
 F 0 "J5" H 9978 5076 50  0000 L CNN
 F 1 "Conn_01x05_Female" H 9978 4985 50  0000 L CNN
-F 2 "Connector_JST:JST_ACH_BM05B-ACHSS-A-GAN-ETF_1x05-1MP_P1.20mm_Vertical" H 9950 5050 50  0001 C CNN
+F 2 "Connector_JST:JST_GH_SM05B-GHS-TB_1x05-1MP_P1.25mm_Horizontal" H 9950 5050 50  0001 C CNN
 F 3 "~" H 9950 5050 50  0001 C CNN
 	1    9950 5050
@@
 Wire Wire Line
 	1550 1950 1550 1850
+$Comp
+L Connector:TestPoint TP2
+U 1 1 5CF55FEB
+P 1150 1100
+F 0 "TP2" H 1208 1218 50  0000 L CNN
+F 1 "TestPoint" H 1208 1127 50  0000 L CNN
+F 2 "TestPoint:TestPoint_THTPad_2.0x2.0mm_Drill1.0mm" H 1350 1100 50  0001 C CNN
+F 3 "~" H 1350 1100 50  0001 C CNN
+	1    1150 1100
+	1    0    0    -1
+$EndComp
+$Comp
+L Connector:Conn_01x05_Female J?
+U 1 1 5CF33BF7
+P 9850 2600
+F 0 "J?" H 9878 2626 50  0000 L CNN
+F 1 "Conn_01x05_Female" H 9878 2535 50  0000 L CNN
+F 2 "Connector_JST:JST_GH_SM05B-GHS-TB_1x05-1MP_P1.25mm_Horizontal" H 9850 2600 50  0001 C CNN
+F 3 "~" H 9850 2600 50  0001 C CNN
+	1    9850 2600
+	1    0    0    -1
+$EndComp
 $EndSCHEMATC
