File: typec2.0/typec2.0.kicad_pcb (KiCad board)
At the start: 2 copper layers, 3 parts, among them U1 TUSB2046, U2 TPS2044-SOIC, U3 SN75240PWR

Commit message: 2.0
Parts:
- added C1: 4.7uf/10V, Capacitor_SMD:C_0603_1608Metric, F.Cu at (138.2, 58.8)
- added C10: 33pf/10V, Capacitor_SMD:C_0201_0603Metric, F.Cu at (149.5, 59.6)
- added C11: 22pf/10V, Capacitor_SMD:C_0201_0603Metric, F.Cu at (149.7, 73.5)
- added C12: 22pf/10V, Capacitor_SMD:C_0201_0603Metric, F.Cu at (148.8, 73.5)
- added C13: 22pf/10V, Capacitor_SMD:C_0201_0603Metric, F.Cu at (153.2, 73.5)
- added C14: 22pf/10V, Capacitor_SMD:C_0201_0603Metric, F.Cu at (152.2, 73.5)
- added C15: 22pf/10V, Capacitor_SMD:C_0201_0603Metric, F.Cu at (159.9, 67.9)
- added C16: 22pf/10V, Capacitor_SMD:C_0201_0603Metric, F.Cu at (158.2, 67.9)
- added C17: 22pf/10V, Capacitor_SMD:C_0201_0603Metric, F.Cu at (158.9, 57.8)
- added C18: 22pf/10V, Capacitor_SMD:C_0201_0603Metric, F.Cu at (160.7, 57.8)
- added C19: 0.1uf/10V, Capacitor_SMD:C_0201_0603Metric, F.Cu at (147.9, 73.4)
- added C2: 22pf/10V, Capacitor_SMD:C_0201_0603Metric, F.Cu at (142.2, 65.6)
- added C20: 0.1uf/10V, Capacitor_SMD:C_0201_0603Metric, F.Cu at (155.0, 71.8)
- added C21: 0.1uf/10V, Capacitor_SMD:C_0201_0603Metric, F.Cu at (156.4, 69.1)
- added C22: 4.7 uf/10 V, Capacitor_SMD:C_0603_1608Metric, F.Cu at (138.2, 56.6)
- added C23: 0.1uf/10V, Capacitor_SMD:C_0201_0603Metric, F.Cu at (156.4, 66.0)
- added C3: 22pf/10V, Capacitor_SMD:C_0201_0603Metric, F.Cu at (144.0, 66.0)
- added C4: 4.7uf/10V, Capacitor_SMD:C_0603_1608Metric, F.Cu at (138.2, 54.7)
- added C5: 4.7uf/10V, Capacitor_SMD:C_0603_1608Metric, F.Cu at (142.5, 55.0)
- added C6: 4.7uf/10V, Capacitor_SMD:C_0603_1608Metric, F.Cu at (147.1, 58.3)
- added C7: 33pf/10V, Capacitor_SMD:C_0201_0603Metric, F.Cu at (149.0, 61.0)
- added C8: 10uf/10V, Capacitor_SMD:C_0603_1608Metric, F.Cu at (145.3, 58.4)
- added C9: 22uf/10V, Capacitor_SMD:C_0603_1608Metric, F.Cu at (140.0, 69.3)
- added D1: RED, LED_SMD:LED_0201_0603Metric, F.Cu at (144.3, 53.7)
- added D2: RED, LED_SMD:LED_0201_0603Metric, F.Cu at (140.2, 54.3)
- added D3: RED, LED_SMD:LED_0201_0603Metric, F.Cu at (147.0, 73.4)
- added D4: RED, LED_SMD:LED_0201_0603Metric, F.Cu at (151.3, 73.5)
- added D5: RED, LED_SMD:LED_0201_0603Metric, F.Cu at (156.4, 70.0)
- added D6: RED, LED_SMD:LED_0201_0603Metric, F.Cu at (156.4, 66.8)
- added D7: RED, LED_SMD:LED_0201_0603Metric, F.Cu at (147.4, 61.0)
- added J1: Conn_01x05_Male, Connector_JST:JST_GH_SM05B-GHS-TB_1x05-1MP_P1.25mm_Horizontal, F.Cu at (135.8, 65.7)
- added J2: Conn_01x05_Female, Connector_JST:JST_GH_SM05B-GHS-TB_1x05-1MP_P1.25mm_Horizontal, F.Cu at (153.7, 85.2)
- added J3: Conn_01x05_Female, Connector_JST:JST_GH_SM05B-GHS-TB_1x05-1MP_P1.25mm_Horizontal, F.Cu at (165.5, 85.2)
- added J4: Conn_01x05_Female, Connector_JST:JST_GH_SM05B-GHS-TB_1x05-1MP_P1.25mm_Horizontal, F.Cu at (165.8, 65.0)
- added J5: Conn_01x05_Female, Connector_JST:JST_GH_SM05B-GHS-TB_1x05-1MP_P1.25mm_Horizontal, F.Cu at (166.0, 53.4)
- added JP1: Jumper_3_Open, Connector_JST:JST_EH_B3B-EH-A_1x03_P2.50mm_Vertical, F.Cu at (166.8, 74.1)
- added JP2: Jumper_3_Open, Connector_JST:JST_EH_B3B-EH-A_1x03_P2.50mm_Vertical, F.Cu at (142.6, 82.0)
- added JP3: Jumper_NO_Small, Connector_JST:JST_EH_B2B-EH-A_1x02_P2.50mm_Vertical, F.Cu at (159.4, 53.5)
- added L1: 1uH/2.1A, Inductor_SMD:L_6.3x6.3_H3, F.Cu at (137.9, 46.0)
- added R1: 22 E, Resistor_SMD:R_0201_0603Metric, F.Cu at (139.6, 66.1)
- added R10: 510 E, Resistor_SMD:R_0201_0603Metric, F.Cu at (158.0, 70.0)
- added R11: 510 E, Resistor_SMD:R_0201_0603Metric, F.Cu at (146.4, 60.9)
- added R12: 22 E, Resistor_SMD:R_0201_0603Metric, F.Cu at (150.5, 73.4)
- added R13: 22 E, Resistor_SMD:R_0201_0603Metric, F.Cu at (147.9, 78.3)
- added R14: 22 E, Resistor_SMD:R_0201_0603Metric, F.Cu at (160.7, 67.8)
- added R15: 22 E, Resistor_SMD:R_0201_0603Metric, F.Cu at (159.0, 67.9)
- added R16: 22 E, Resistor_SMD:R_0201_0603Metric, F.Cu at (157.8, 79.7)
- added R17: 22 E, Resistor_SMD:R_0201_0603Metric, F.Cu at (157.9, 77.6)
- added R18: 22 E, Resistor_SMD:R_0201_0603Metric, F.Cu at (157.2, 57.8)
- added R19: 22 E, Resistor_SMD:R_0201_0603Metric, F.Cu at (159.8, 57.8)
- added R2: 22 E, Resistor_SMD:R_0201_0603Metric, F.Cu at (139.6, 64.1)
- added R20: 15 K, Resistor_SMD:R_0201_0603Metric, F.Cu at (150.1, 47.2)
- added R21: 15 K, Resistor_SMD:R_0201_0603Metric, F.Cu at (155.4, 47.1)
- added R22: 15 K, Resistor_SMD:R_0201_0603Metric, F.Cu at (147.5, 47.0)
- added R23: 15 K, Resistor_SMD:R_0201_0603Metric, F.Cu at (152.5, 47.2)
- added R24: 15 K, Resistor_SMD:R_0201_0603Metric, F.Cu at (146.5, 47.0)
- added R25: 15 K, Resistor_SMD:R_0201_0603Metric, F.Cu at (149.2, 47.2)
- added R26: 15 K, Resistor_SMD:R_0201_0603Metric, F.Cu at (151.4, 47.2)
- added R27: 15 K, Resistor_SMD:R_0201_0603Metric, F.Cu at (156.5, 47.2)
- added R3: 510 E, Resistor_SMD:R_0201_0603Metric, F.Cu at (144.5, 55.0)
- added R4: 178 K, Resistor_SMD:R_0201_0603Metric, F.Cu at (138.5, 50.0)
- added R5: 1.5 K, Resistor_SMD:R_0201_0603Metric, F.Cu at (150.0, 61.0)
- added R6: 510 E, Resistor_SMD:R_0201_0603Metric, F.Cu at (140.2, 51.3)
- added R7: 510 E, Resistor_SMD:R_0201_0603Metric, F.Cu at (147.4, 74.9)
- added R8: 510 E, Resistor_SMD:R_0201_0603Metric, F.Cu at (151.1, 74.9)
- added R9: 510 E, Resistor_SMD:R_0201_0603Metric, F.Cu at (156.7, 71.4)
- added TP1: TestPoint, TestPoint:TestPoint_THTPad_2.0x2.0mm_Drill1.0mm, F.Cu at (142.5, 51.7)
- added TP2: TestPoint, TestPoint:TestPoint_THTPad_2.0x2.0mm_Drill1.0mm, F.Cu at (134.6, 58.6)
- added U4: TPS62082-WSON, TPS62081-WSON:TPS62082-WSON, F.Cu at (138.4, 52.4)
- added U5: SN75240PWR, SN75240PWR:SN75240PWR, F.Cu at (142.9, 61.2)
- added U6: SN75240PWR, SN75240PWR:SN75240PWR, F.Cu at (153.4, 78.9)
- added U7: SN75240PWR, SN75240PWR:SN75240PWR, F.Cu at (159.3, 62.9)
- added Y1: Crystal, Crystal:Crystal_HC49-U_Vertical, F.Cu at (165.5, 43.6)
- moved U3 154.8 mm to (150.6, 43.6)
- moved U1 133.5 mm to (150.3, 67.5)
- moved U2 127.2 mm to (150.9, 52.6), turned to 90 degrees
Connections:
- U1 pad 1: (no net) -> Net-(C2-Pad2)
- U1 pad 10: (no net) -> Net-(C19-Pad2)
- U1 pad 11: (no net) -> Net-(C12-Pad2)
- U1 pad 12: (no net) -> Net-(C11-Pad2)
- U1 pad 13: (no net) -> Net-(D4-Pad1)
- U1 pad 14: (no net) -> Net-(C20-Pad2)
- U1 pad 15: (no net) -> Net-(C14-Pad2)
- U1 pad 16: (no net) -> Net-(C13-Pad2)
- U1 pad 17: (no net) -> Net-(D5-Pad1)
- U1 pad 18: (no net) -> Net-(C21-Pad2)
- U1 pad 19: (no net) -> Net-(C16-Pad2)
- U1 pad 2: (no net) -> Net-(C3-Pad2)
- U1 pad 20: (no net) -> Net-(C15-Pad2)
- U1 pad 21: (no net) -> Net-(D6-Pad1)
- U1 pad 22: (no net) -> Net-(C21-Pad2)
- U1 pad 23: (no net) -> Net-(C18-Pad2)
- U1 pad 24: (no net) -> Net-(C17-Pad2)
- U1 pad 25: (no net) -> Vout(3.3V)
- U1 pad 26: (no net) -> Net-(JP1-Pad2)
- U1 pad 27: (no net) -> GND
- U1 pad 28: (no net) -> GND
- U1 pad 29: (no net) -> Net-(C7-Pad2)
- U1 pad 3: (no net) -> Vout(3.3V)
- U1 pad 30: (no net) -> Net-(C7-Pad2)
- U1 pad 31: (no net) -> GND
- U1 pad 32: (no net) -> SUSPND
- U1 pad 4: (no net) -> Net-(JP2-Pad2)
- U1 pad 7: (no net) -> GND
- U1 pad 8: (no net) -> GND
- U1 pad 9: (no net) -> Net-(D3-Pad1)
- U2 pad 1: (no net) -> GND
- U2 pad 10: (no net) -> VOUT4(5V)
- U2 pad 11: (no net) -> VOUT3(5V)
- U2 pad 12: (no net) -> Net-(R23-Pad1)
- U2 pad 13: (no net) -> Net-(R20-Pad1)
- U2 pad 14: (no net) -> VOUT2(5V)
- U2 pad 15: (no net) -> VOUT1(5V)
- U2 pad 16: (no net) -> Net-(R22-Pad1)
- U2 pad 2: (no net) -> VBUS(5V)
- U2 pad 3: (no net) -> Net-(D3-Pad1)
- U2 pad 4: (no net) -> Net-(D4-Pad1)
- U2 pad 5: (no net) -> GND
- U2 pad 6: (no net) -> VBUS(5V)
- U2 pad 7: (no net) -> Net-(D5-Pad1)
- U2 pad 8: (no net) -> Net-(D6-Pad1)
- U2 pad 9: (no net) -> Net-(R21-Pad2)
- U3 pad 1: (no net) -> GND
- U3 pad 2: (no net) -> Net-(R22-Pad1)
- U3 pad 3: (no net) -> GND
- U3 pad 4: (no net) -> Net-(R20-Pad1)
- U3 pad 5: (no net) -> GND
- U3 pad 6: (no net) -> Net-(R23-Pad1)
- U3 pad 7: (no net) -> GND
- U3 pad 8: (no net) -> Net-(R21-Pad2)
Routing:
- net GND: track 0.00 -> 270.3 mm, vias 0 -> 5
- net VBUS(5V): track 0.00 -> 101.7 mm
- net Vout(3.3V): track 0.00 -> 77.6 mm, vias 0 -> 2
- net VOUT2(5V): track 0.00 -> 38.7 mm, vias 0 -> 2
- net VOUT1(5V): track 0.00 -> 35.4 mm, vias 0 -> 2
- net Net-(C20-Pad2): track 0.00 -> 30.2 mm, vias 0 -> 2
- net VOUT(3.3V): track 0.00 -> 29.3 mm, vias 0 -> 3
- net Net-(C7-Pad2): track 0.00 -> 28.8 mm, vias 0 -> 1
- net Net-(JP3-Pad1): track 0.00 -> 28.6 mm, vias 0 -> 2
- net VOUT3(5V): track 0.00 -> 28.1 mm, vias 0 -> 1
- net Net-(C19-Pad2): track 0.00 -> 26.9 mm, vias 0 -> 2
- net Net-(C21-Pad2): track 0.00 -> 26.1 mm, vias 0 -> 2
- net Net-(C10-Pad1): track 0.00 -> 21.6 mm, vias 0 -> 1
- net Net-(D4-Pad1): track 0.00 -> 19.4 mm, vias 0 -> 2
- net Net-(D3-Pad1): track 0.00 -> 19.0 mm, vias 0 -> 2
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Other:
- copper layers 2 -> 4
